File: 2ndKeyboard/matrix_sch.kicad_sch (KiCad schematic)
At the start: 174 parts, among them K1 KEYSW, K10 KEYSW, K11 KEYSW, K12 KEYSW, K13 KEYSW, K14 KEYSW, K15 KEYSW, K16 KEYSW, K17 KEYSW, K18 KEYSW, K19 KEYSW, K2 KEYSW, K20 KEYSW, K21 KEYSW, K22 KEYSW, K23 KEYSW, K24 KEYSW, K25 KEYSW, K26 KEYSW, K27 KEYSW, K28 KEYSW, K29 KEYSW, K3 KEYSW, K30 KEYSW, K31 KEYSW, K32 KEYSW, K33 KEYSW, K34 KEYSW, K35 KEYSW, K36 KEYSW, K37 KEYSW, K38 KEYSW, K39 KEYSW, K4 KEYSW, K40 KEYSW, K41 KEYSW, K42 KEYSW, K43 KEYSW, K44 KEYSW, K45 KEYSW, K46 KEYSW, K47 KEYSW, K48 KEYSW, K49 KEYSW, K5 KEYSW, K50 KEYSW, K51 KEYSW, K52 KEYSW, K53 KEYSW, K54 KEYSW, K55 KEYSW, K56 KEYSW, K57 KEYSW, K58 KEYSW, K59 KEYSW, K6 KEYSW, K60 KEYSW, K61 KEYSW, K62 KEYSW, K63 KEYSW, K64 KEYSW, K65 KEYSW, K66 KEYSW, K67 KEYSW, K68 KEYSW, K69 KEYSW, K7 KEYSW, K70 KEYSW, K71 KEYSW, K72 KEYSW, K73 KEYSW, K74 KEYSW, K75 KEYSW, K76 KEYSW, K77 KEYSW, K78 KEYSW, K79 KEYSW, K8 KEYSW, K80 KEYSW, K81 KEYSW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

Commit message: schematic.2
Parts:
- K1: value KEYSW -> ESC
- K10: value KEYSW -> F9
- K11: value KEYSW -> F10
- K12: value KEYSW -> F11
- K13: value KEYSW -> F12
- K14: value KEYSW -> Imp_Ecran
- K15: value KEYSW -> Defilement
- K16: value KEYSW -> Pause
- K17: value KEYSW -> /
- K18: value KEYSW -> 1
- K19: value KEYSW -> 2
- K2: value KEYSW -> F!
- K20: value KEYSW -> 3
- K21: value KEYSW -> 4
- K22: value KEYSW -> 5
- K23: value KEYSW -> 6
- K24: value KEYSW -> 7
- K25: value KEYSW -> 8
- K26: value KEYSW -> 9
- K27: value KEYSW -> 0
- K28: value KEYSW -> -
- K29: value KEYSW -> =
- K3: value KEYSW -> F2
- K31: value KEYSW -> Ins
- K32: value KEYSW -> Debut
- K33: value KEYSW -> Next
- K34: value KEYSW -> TAB
- K35: value KEYSW -> Q
- K36: value KEYSW -> W
- K37: value KEYSW -> E
- K38: value KEYSW -> R
- K39: value KEYSW -> T
- K4: value KEYSW -> F3
- K40: value KEYSW -> Y
- K41: value KEYSW -> U
- K42: value KEYSW -> I
- K43: value KEYSW -> O
- K44: value KEYSW -> P
- K45: value KEYSW -> ^
- K46: value KEYSW -> Ç
- K47: value KEYSW -> À
- K48: value KEYSW -> Suppr
- K49: value KEYSW -> FIN
- K5: value KEYSW -> F4
- K50: value KEYSW -> Previous
- K51: value KEYSW -> CAPS LOCK
- K52: value KEYSW -> A
- K53: value KEYSW -> S
- K54: value KEYSW -> D
- K55: value KEYSW -> F
- K56: value KEYSW -> G
- K57: value KEYSW -> H
- K58: value KEYSW -> J
- K59: value KEYSW -> K
- K6: value KEYSW -> F5
- K60: value KEYSW -> L
- K61: value KEYSW -> ;
- K62: value KEYSW -> È
- K63: value KEYSW -> ENTER
- K64: value KEYSW -> MAJ G.
- K65: value KEYSW -> Z
- K66: value KEYSW -> X
- K67: value KEYSW -> C
- K68: value KEYSW -> V
- K69: value KEYSW -> B
- K7: value KEYSW -> F6
- K70: value KEYSW -> N
- K71: value KEYSW -> M
- K72: value KEYSW -> ,
- K73: value KEYSW -> .
- K74: value KEYSW -> É
- K75: value KEYSW -> MAJ D.
- K76: value KEYSW -> UP Arrow
- K77: value KEYSW -> CTRL G.
- K78, K82: value KEYSW -> WINDOWS
- K79: value KEYSW -> ALT G.
- K8: value KEYSW -> F7
- K80: value KEYSW -> BARRE
- K81: value KEYSW -> ALT D.
- K83: value KEYSW -> MENU
- K84: value KEYSW -> CTRL D.
- K85: value KEYSW -> LEFT Arrow
- K86: value KEYSW -> DOWN Arrow
- K87: value KEYSW -> RIGHT Arrow
- K9: value KEYSW -> F8

Commit message: pcb
Parts:
- D1, D10, D11, D12, D13, D14, D15, D16, D17, D18, D19, D2, D20, D21, D22, D23, D24, D25, D26, D27, D28, D29, D3, D30, D31, D32, D33, D34, D35, D36, D37, D38, D39, D4, D40, D41, D42, D43, D44, D45, D46, D47, D48, D49, D5, D50, D51, D52, D53, D54, D55, D56, D57, D58, D59, D6, D60, D61, D62, D63, D64, D65, D66, D67, D68, D69, D7, D70, D71, D72, D73, D74, D75, D76, D77, D78, D79, D8, D80, D81, D82, D83, D84, D85, D86, D87, D9: footprint Diode_SMD:D_0805_2012Metric_Pad1.15x1.40mm_HandSolder -> Diode_SMD:D_SOD-123
- K2: value F! -> F1
